Commit message: viz/aira: URDF piatto rigenerato con busto+testa (per RViz del controller)
Co-Authored-By: Claude Opus 4.8 (1M context) <noreply@anthropic.com>

File: viz/aira/aira_base.urdf (robot description, URDF)
Before this commit: robot aira_base, 8 links, 7 joints
Links:
- added link camera_link; visual box size=0.03 0.075 0.03
- added link head_link, mass 0.6; collision box size=0.12 0.12 0.14; visual box size=0.12 0.12 0.14
- added link head_pan_link, mass 0.05
- added link head_tilt_link, mass 0.05
- added link mast_link, mass 1.0; collision box size=0.04 0.04 0.5; visual box size=0.04 0.04 0.5
- added link neck_link, mass 0.1; visual cylinder length=0.06 radius=0.02
- added link torso_link, mass 2.0; collision box size=0.14 0.18 0.3; visual box size=0.14 0.18 0.3
- added link torso_pitch_link, mass 0.05
Joints:
- added joint camera_joint: type fixed, parent head_link, child camera_link, origin xyz=0.06 0 0.084 rpy=0 0 0
- added joint head_pan: type revolute, parent neck_link, child head_pan_link, origin xyz=0 0 0.06 rpy=0 0 0, axis 0 0 1, limit lower=-1.5707963267948966 upper=1.5707963267948966 effort=10 velocity=3.0
- added joint head_pitch: type revolute, parent head_tilt_link, child head_link, origin xyz=0 0 0 rpy=0 0 0, axis 0 1 0, limit lower=-0.7853981633974483 upper=0.7853981633974483 effort=10 velocity=3.0
- added joint head_tilt: type revolute, parent head_pan_link, child head_tilt_link, origin xyz=0 0 0 rpy=0 0 0, axis 1 0 0, limit lower=-0.7853981633974483 upper=0.7853981633974483 effort=10 velocity=3.0
- added joint mast_joint: type fixed, parent base_link, child mast_link, origin xyz=0 0 0 rpy=0 0 0
- added joint neck_joint: type fixed, parent torso_link, child neck_link, origin xyz=0 0 0.3 rpy=0 0 0
- added joint torso_pitch: type revolute, parent mast_link, child torso_pitch_link, origin xyz=0 0 0.5 rpy=0 0 0, axis 0 1 0, limit lower=-0.5235987755982988 upper=0.7853981633974483 effort=80 velocity=2.0
- added joint torso_tilt: type revolute, parent torso_pitch_link, child torso_link, origin xyz=0 0 0 rpy=0 0 0, axis 1 0 0, limit lower=-0.4363323129985824 upper=0.4363323129985824 effort=80 velocity=2.0
